Commit message: Added launch

File: my_ur5e_moveit_config/config/my_ur5e.ros2_control.xacro (robot description, xacro)
@@ -2,5 +2,5 @@
 <robot xmlns:xacro="http://www.ros.org/wiki/xacro">
     <xacro:macro name="my_ur5e_ros2_control" params="name initial_positions_file">
-        <xacro:property name="initial_positions" value="${load_yaml(initial_positions_file)['initial_positions']}"/>
+        <xacro:property name="initial_positions" value="${xacro.load_yaml(initial_positions_file)['initial_positions']}"/>
         <ros2_control name="${name}" type="system">
             <hardware>

File: my_ur5e_moveit_config/config/my_ur5e.urdf.xacro (robot description, xacro)
@@ -1,13 +1,9 @@
 <?xml version="1.0"?>
 <robot xmlns:xacro="http://www.ros.org/wiki/xacro" name="my_ur5e">
-<!-- Lines removed by Gerard
     <xacro:arg name="initial_positions_file" default="initial_positions.yaml" />
--->
     <!-- Import my_ur5e urdf file -->
     <xacro:include filename="$(find my_ur5e_description)/urdf/ur.urdf.xacro" />
     <!-- Import control_xacro -->
     <xacro:include filename="my_ur5e.ros2_control.xacro" />
-<!-- Lines removed by gerard
     <xacro:my_ur5e_ros2_control name="FakeSystem" initial_positions_file="$(arg initial_positions_file)"/>
--->
 </robot>

Commit message: 20231023

File: my_ur5e_moveit_config/config/my_ur5e.ros2_control.xacro (robot description, xacro)
@@ -2,5 +2,5 @@
 <robot xmlns:xacro="http://www.ros.org/wiki/xacro">
     <xacro:macro name="my_ur5e_ros2_control" params="name initial_positions_file">
-        <xacro:property name="initial_positions" value="${xacro.load_yaml(initial_positions_file)['initial_positions']}"/>
+        <xacro:property name="initial_positions" value="${load_yaml(initial_positions_file)['initial_positions']}"/>
         <ros2_control name="${name}" type="system">
             <hardware>
